File: USBPD-2/USBPD-2.kicad_sch (KiCad schematic)
At the start: 122 parts, among them J1 USB_C_Receptacle_USB2.0_14P, J2 USB_C_Receptacle_USB2.0_14P, J3 Screw_Terminal_01x05, Q1 DMT6008LFG, Q2 DMT6008LFG, Q3 DMT6008LFG, U1 LM74700, U2 TPS55289RYQR, U3 TPS55289RYQR, U4 TPS70950DBVR, U5 AP43776, U6 SLM2009

Commit message: Modularized kicad schematic
Parts:
- added J10, J12, J4, J5, J6, J7, J8, J9: Conn_01x01_Pin, symbol Connector:Conn_01x01_Pin
- added J11, J14: Conn_01x02_Pin, symbol Connector:Conn_01x02_Pin
- added J13: Conn_01x04_Pin, symbol Connector:Conn_01x04_Pin
Connections:
- net GND: now also J13.4 (Pin_4)
- net SW: now also L2.2; no longer L2.1
- net VCC: now also J13.1 (Pin_1)
- removed net BUCK_OUT: C10.1, C28.1, C30.1, C31.1, C34.1, C6.1, C7.1, C8.1, C9.1, L2.2, R15.1, R28.1, R3.1, U2.7 (VIN), U3.7 (VIN)
- net PWR_IN renamed ENABLE_IN
- net ENABLE_IN: now also J5.1 (Pin_1); no longer C52.1, D13.2 (A2), J3.1 (Pin_1)
- net Q_PRIM renamed QPRIM_OUT
- net QPRIM_OUT: now also J13.2 (Pin_2); no longer Q1.4 (G)
- net Q_SYNC renamed QPRIM_IN
- net QPRIM_IN: now also J14.2 (Pin_2); no longer U6.5 (LO)
- new net BOOST_IN: C5.1, J7.1 (Pin_1), L2.1
- new net BOOST_OUT: C6.1, J8.1 (Pin_1), Q1.5 (D)
- new net CONVA_IN: C10.1, C7.1, C8.1, C9.1, J9.1 (Pin_1), R3.1, U2.7 (VIN)
- new net CONVB_IN: C28.1, C30.1, C31.1, C34.1, J10.1 (Pin_1), R15.1, U3.7 (VIN)
- new net ENABLE_OUT: J6.1 (Pin_1), L1.2
- new net PWR_OUT: C52.1, D13.2 (A2), J3.1 (Pin_1), J4.1 (Pin_1)
- new net QSYNC_IN: J14.1 (Pin_1), Q1.4 (G)
- new net QSYNC_OUT: J13.3 (Pin_3), U6.5 (LO)
- new net SPLITTER: J11.1 (Pin_1), J11.2 (Pin_2), J12.1 (Pin_1), R28.1
Other:
- note added: "Boost Converter"
- note added: "GPIO1"
- note removed: "Buck Converter"
- moved on the sheet: C1, C10, C11, C12, C13, C14, C15, C16, C17, C18, C19, C2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

Commit message: 11/11 changes
Parts:
- removed C5, C6: 68u/35V, symbol Device:C_Polarized_US
- removed J13: Conn_01x04_Pin, symbol Connector:Conn_01x04_Pin
- removed J14: Conn_01x02_Pin, symbol Connector:Conn_01x02_Pin
- removed J3: Screw_Terminal_01x05, symbol Connector:Screw_Terminal_01x05
- added C5, C55, C56, C6: 100n, symbol Device:C
- added C57, C58, C59, C60: 1n, symbol Device:C
- added C61, C62: 2u2, symbol Device:C
- added C63, C64: C_Polarized_US, symbol Device:C_Polarized_US
- added D15: VCC, symbol Device:LED
- added J15: Conn_01x08_Pin, symbol Connector:Conn_01x08_Pin
- added J16: Conn_01x04_Pin, symbol Connector:Conn_01x04_Pin
- added J3: Power Terminal, symbol Connector:Screw_Terminal_01x04
- added Q4: DMT6008LFG, Package_SON:Diodes_PowerDI3333-8, symbol Transistor_FET:DMT6008LFG
- added R35, R37, R39, R41: 450k, symbol Device:R
- added R36, R38, R40, R42: 50k, symbol Device:R
- added R43: 698R, symbol Device:R
- added U10, U7, U8, U9: ACS712ELCTR-20A-T, Package_SO:SOIC-8_3.9x4.9mm_P1.27mm, symbol USBPD-2:ACS712
- added U11: ADC128S102CIMTX/NOPB, USBPD-2:ADC128, symbol USBPD-2:ADC128
- added U12: TPS70933, USBPD-2:TPS709, symbol USBPD-2:TPS709
- L2: value 10u -> L_Iron
- U4: value TPS70950DBVR -> TPS70950; footprint (none) -> USBPD-2:TPS709
- U5: value AP43776 -> AP43776QZDZW20-13; footprint (none) -> USBPD-2:AP43776
- U6: value SLM2009 -> SLM2009CA-DG; footprint (none) -> USBPD-2:SLM2009
Connections:
- net QSYNC_IN is gone; now on net QPRIM: Q1.4 (G)
- net QSYNC_OUT is gone; now on net QSYNC: U6.5 (LO)
- net BATTERY: now also J3.3 (Pin_3), Q4.5 (D); no longer C49.1, U4.1 (IN), U4.3 (EN)
- net GND: now also C5.2, C55.2, C56.2, C57.2, C58.2, C59.2, C6.2, C60.2, C61.2, C62.2, C63.2, C64.2, D15.1 (K), J3.2 (Pin_2), J3.4 (Pin_4), R36.2, R38.2, R40.2, R42.2, U10.5 (GND), U11.12 (DGND), U11.3 (AGND), U12.2 (GND), U7.5 (GND), U8.5 (GND), U9.5 (GND)
- net PWR_OUT: now also J3.1 (Pin_1)
- net VCC: now also C5.1, C55.1, C56.1, C6.1, U10.8 (VCC), U11.2 (VA), U7.8 (VCC), U8.8 (VCC), U9.8 (VCC); no longer C53.1, D14.2 (A), U6.1 (VCC)
- net BOOST_IN renamed BUCK_IN
- net BUCK_IN: now also C63.1
- net BOOST_OUT: no longer names the net of Q1.5 (D)
- net BOOST_OUT: now also L2.2; no longer J8.1 (Pin_1)
- net QPRIM_IN renamed QSYNC
- net QPRIM_OUT renamed QPRIM
- net SW renamed BUCK_OUT
- net BUCK_OUT: now also J8.1 (Pin_1), C64.1; no longer L2.2
- new net: J15.3 (Pin_3), R37.1, U8.1 (IP+), U8.2 (IP+)
- new net: C58.1, U8.6 (FILTER)
- new net: C57.1, U7.6 (FILTER)
- new net: D15.2 (A), R43.2
- new net: C53.1, D14.2 (A), U6.1 (VCC)
- new net: J15.1 (Pin_1), R35.1, U7.1 (IP+), U7.2 (IP+)
- new net: J15.2 (Pin_2), U7.3 (IP-), U7.4 (IP-)
- new net: J15.4 (Pin_4), U8.3 (IP-), U8.4 (IP-)
- new net: J15.5 (Pin_5), R39.1, U9.1 (IP+), U9.2 (IP+)
- new net: J15.6 (Pin_6), U9.3 (IP-), U9.4 (IP-)
- new net: J15.7 (Pin_7), R41.1, U10.1 (IP+), U10.2 (IP+)
- new net: J15.8 (Pin_8), U10.3 (IP-), U10.4 (IP-)
- new net: C60.1, U10.6 (FILTER)
- new net: C59.1, U9.6 (FILTER)
- new net 12V: C49.1, C61.1, Q4.1 (S), Q4.2 (S), Q4.3 (S), U12.1 (IN), U12.3 (EN), U4.1 (IN), U4.3 (EN)
- new net Isens1: U11.5 (IN1), U7.7 (VIOUT)
- new net Isens2: U11.7 (IN3), U8.7 (VIOUT)
- new net Isens3: U11.9 (IN5), U9.7 (VIOUT)
- new net Isens4: U10.7 (VIOUT), U11.11 (IN7)
- new net MISO: J16.3 (Pin_3), U11.15 (MISO)
- new net MOSI: J16.4 (Pin_4), U11.14 (MOSI)
- new net SCLK: J16.2 (Pin_2), U11.16 (SCLK)
- new net VDD: C62.1, R43.1, U11.13 (VD), U12.5 (OUT)
- new net Vsens1: R35.2, R36.1, U11.4 (IN0)
- new net Vsens2: R37.2, R38.1, U11.6 (IN2)
- new net Vsens3: R39.2, R40.1, U11.8 (IN4)
- new net Vsens4: R41.2, R42.1, U11.10 (IN6)
- new net /CS: J16.1 (Pin_1), U11.1 (/CS)
Other:
- note added: "12V Battery"
- note added: "15V Vbr TVS Diodes (SMAJ13CA)"
- note added: "3.3V out"
- note added: "5.0V out"
- note added: "50V Vbr TVS Diode (SMAJ45CA)"
- note added: "ACS712ELCTR-20A-T Current sense"
- note added: "Assuming a 50V upper limit, VA=5V, Vsens should be 10% of IP voltage Higher = 9 * Lower"
- note added: "Buck Converter"
- note added: "Buck out"
- note added: "Conv A and B in"
- note added: "Power Supply"
- note added: "Resistor tolerances should be ≤ ±1%"
- note added: "Sensing"
- note removed: "Battery should be 4x 1.5V AA or AAA"
- note removed: "Boost Converter"
- note removed: "Gate Driver"
- note removed: "LDO Power Supply (2.7-32V input)"
- moved on the sheet: C1, C2, C3, C4, C49, C50, C52, C53, C54, D1, D13, D14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

Commit message: rev1_idle_mangement
Parts:
- added 5.1V: D_Zener, symbol Device:D_Zener
- added C65: 100uF, symbol Device:C
- added D17: D, symbol Device:D
- added Q5: DMT6008LFG, Package_SON:Diodes_PowerDI3333-8, symbol Transistor_FET:DMT6008LFG
- added R44: 450k, symbol Device:R
- added R45: 50k, symbol Device:R
- added R46: 60 kOhms, symbol Device:R
Connections:
- net 12V: now also Q5.5 (D)
- net GND: now also 5.1V.2 (A), R45.2, R46.2
- net Vsens1: now also 5.1V.1 (K), D17.2 (A), R44.2, R45.1
- new net: C65.2, R46.1
- new net: C65.1, D17.1 (K), Q5.4 (G)
- new net 1: R44.1
- new net 12 V BUS: Q5.1 (S), Q5.2 (S), Q5.3 (S)
Other:
- note added: "LV Power Management"
